File: PCB/TaggerMainboard/TaggerMainboard.sch (KiCad schematic (older format))
At the start: 80 parts

Commit message: Footprints für Anschlüsse hinterlegt
Parts:
- J?: footprint (none) -> Connector_PinHeader_2.54mm:PinHeader_2x03_P2.54mm_Vertical
- J? (x6): footprint (none) -> Connector_JST:JST_PH_B2B-PH-K_1x02_P2.00mm_Vertical
- J? (x2): footprint (none) -> Connector_JST:JST_PH_B3B-PH-K_1x03_P2.00mm_Vertical
- J? (x2): footprint (none) -> Connector_JST:JST_PH_B4B-PH-K_1x04_P2.00mm_Vertical
- J? (x2): footprint (none) -> Connector_JST:JST_PH_B7B-PH-K_1x07_P2.00mm_Vertical
- J?: footprint (none) -> Connector_JST:JST_PH_B6B-PH-K_1x06_P2.00mm_Vertical
Changed lines of the file:
@@
 EESchema Schematic File Version 4
-LIBS:ProTagger-cache
 EELAYER 26 0
 EELAYER END
@@
 F 0 "J?" H 13350 5617 50  0000 C CNN
 F 1 "ICSP" H 13350 5526 50  0000 C CNN
-F 2 "" H 13300 5300 50  0001 C CNN
+F 2 "Connector_PinHeader_2.54mm:PinHeader_2x03_P2.54mm_Vertical" H 13300 5300 50  0001 C CNN
 F 3 "~" H 13300 5300 50  0001 C CNN
 	1    13300 5300
@@
 F 0 "J?" H 13579 892 50  0000 L CNN
 F 1 "JST_PH_Trigger" H 13579 801 50  0000 L CNN
-F 2 "" H 13500 900 50  0001 C CNN
+F 2 "Connector_JST:JST_PH_B2B-PH-K_1x02_P2.00mm_Vertical" H 13500 900 50  0001 C CNN
 F 3 "~" H 13500 900 50  0001 C CNN
 	1    13500 900
@@
 F 0 "J?" H 15180 892 50  0000 L CNN
 F 1 "JST_PH_Reload" H 15180 801 50  0000 L CNN
-F 2 "" H 15100 900 50  0001 C CNN
+F 2 "Connector_JST:JST_PH_B2B-PH-K_1x02_P2.00mm_Vertical" H 15100 900 50  0001 C CNN
 F 3 "~" H 15100 900 50  0001 C CNN
 	1    15100 900
@@
 F 0 "J?" H 13580 1742 50  0000 L CNN
 F 1 "JST_PH_Info" H 13580 1651 50  0000 L CNN
-F 2 "" H 13500 1750 50  0001 C CNN
+F 2 "Connector_JST:JST_PH_B2B-PH-K_1x02_P2.00mm_Vertical" H 13500 1750 50  0001 C CNN
 F 3 "~" H 13500 1750 50  0001 C CNN
 	1    13500 1750
@@
 F 0 "J?" H 15179 1742 50  0000 L CNN
 F 1 "JST_PH_Special" H 15179 1651 50  0000 L CNN
-F 2 "" H 15100 1750 50  0001 C CNN
+F 2 "Connector_JST:JST_PH_B2B-PH-K_1x02_P2.00mm_Vertical" H 15100 1750 50  0001 C CNN
 F 3 "~" H 15100 1750 50  0001 C CNN
 	1    15100 1750
@@
 F 0 "J?" H 13530 2792 50  0000 L CNN
 F 1 "JST_PH_LEDbar_right" H 13530 2701 50  0000 L CNN
-F 2 "" H 13450 2750 50  0001 C CNN
+F 2 "Connector_JST:JST_PH_B3B-PH-K_1x03_P2.00mm_Vertical" H 13450 2750 50  0001 C CNN
 F 3 "~" H 13450 2750 50  0001 C CNN
 	1    13450 2750
@@
 F 0 "J?" H 15179 2792 50  0000 L CNN
 F 1 "JST_PH_LEDbar_left" H 15179 2701 50  0000 L CNN
-F 2 "" H 15100 2750 50  0001 C CNN
+F 2 "Connector_JST:JST_PH_B3B-PH-K_1x03_P2.00mm_Vertical" H 15100 2750 50  0001 C CNN
 F 3 "~" H 15100 2750 50  0001 C CNN
 	1    15100 2750
@@
 F 0 "J?" H 15180 3442 50  0000 L CNN
 F 1 "JSP_PH_Sensor" H 15180 3351 50  0000 L CNN
-F 2 "" H 15100 3450 50  0001 C CNN
+F 2 "Connector_JST:JST_PH_B4B-PH-K_1x04_P2.00mm_Vertical" H 15100 3450 50  0001 C CNN
 F 3 "~" H 15100 3450 50  0001 C CNN
 	1    15100 3450
@@
 F 0 "J?" H 13530 3442 50  0000 L CNN
 F 1 "JSP_PH_Sensor" H 13530 3351 50  0000 L CNN
-F 2 "" H 13450 3450 50  0001 C CNN
+F 2 "Connector_JST:JST_PH_B4B-PH-K_1x04_P2.00mm_Vertical" H 13450 3450 50  0001 C CNN
 F 3 "~" H 13450 3450 50  0001 C CNN
 	1    13450 3450
@@
 F 0 "J?" H 15180 4442 50  0000 L CNN
 F 1 "JST_PH_Keypad" H 15180 4351 50  0000 L CNN
-F 2 "" H 15100 4400 50  0001 C CNN
+F 2 "Connector_JST:JST_PH_B7B-PH-K_1x07_P2.00mm_Vertical" H 15100 4400 50  0001 C CNN
 F 3 "~" H 15100 4400 50  0001 C CNN
 	1    15100 4400
@@
 F 0 "J?" H 15180 5842 50  0000 L CNN
 F 1 "JST_PH_Display" H 15180 5751 50  0000 L CNN
-F 2 "" H 15100 5800 50  0001 C CNN
+F 2 "Connector_JST:JST_PH_B7B-PH-K_1x07_P2.00mm_Vertical" H 15100 5800 50  0001 C CNN
 F 3 "~" H 15100 5800 50  0001 C CNN
 	1    15100 5800
@@
 F 0 "J?" H 8429 5992 50  0000 L CNN
 F 1 "JST_PH_Speaker" H 8429 5901 50  0000 L CNN
-F 2 "" H 8350 6000 50  0001 C CNN
+F 2 "Connector_JST:JST_PH_B2B-PH-K_1x02_P2.00mm_Vertical" H 8350 6000 50  0001 C CNN
 F 3 "~" H 8350 6000 50  0001 C CNN
 	1    8350 6000
@@
 F 0 "J?" H 10580 8592 50  0000 L CNN
 F 1 "Conn_01x06" H 10580 8501 50  0000 L CNN
-F 2 "" H 10500 8600 50  0001 C CNN
+F 2 "Connector_JST:JST_PH_B6B-PH-K_1x06_P2.00mm_Vertical" H 10500 8600 50  0001 C CNN
 F 3 "~" H 10500 8600 50  0001 C CNN
 	1    10500 8600
@@
 F 0 "J?" H 10320 3275 50  0000 C CNN
 F 1 "Conn_01x02" H 10320 3366 50  0000 C CNN
-F 2 "" H 10400 3600 50  0001 C CNN
+F 2 "Connector_JST:JST_PH_B2B-PH-K_1x02_P2.00mm_Vertical" H 10400 3600 50  0001 C CNN
 F 3 "~" H 10400 3600 50  0001 C CNN
 	1    10400 3600

Commit message: LED + Kondensatoren (keine CP) mit Footprint hinterlegt
Parts:
- C? (x11): footprint (none) -> Capacitor_SMD:C_0805_2012Metric
- D? (x3): footprint (none) -> LED_SMD:LED_1206_3216Metric
Changed lines of the file:
@@
 F 0 "C?" H 1692 2296 50  0000 L CNN
 F 1 "100nF" H 1600 2200 50  0000 L CNN
-F 2 "" H 1600 2250 50  0001 C CNN
+F 2 "Capacitor_SMD:C_0805_2012Metric" H 1600 2250 50  0001 C CNN
 F 3 "~" H 1600 2250 50  0001 C CNN
 	1    1600 2250
@@
 F 0 "C?" H 1342 2296 50  0000 L CNN
 F 1 "100nF" H 1250 2200 50  0000 L CNN
-F 2 "" H 1250 2250 50  0001 C CNN
+F 2 "Capacitor_SMD:C_0805_2012Metric" H 1250 2250 50  0001 C CNN
 F 3 "~" H 1250 2250 50  0001 C CNN
 	1    1250 2250
@@
 F 0 "C?" H 992 2296 50  0000 L CNN
 F 1 "100nF" H 900 2200 50  0000 L CNN
-F 2 "" H 900 2250 50  0001 C CNN
+F 2 "Capacitor_SMD:C_0805_2012Metric" H 900 2250 50  0001 C CNN
 F 3 "~" H 900 2250 50  0001 C CNN
 	1    900  2250
@@
 F 0 "C?" H 1550 1800 50  0000 L CNN
 F 1 "100nF" H 1550 1700 50  0000 L CNN
-F 2 "" H 1500 1750 50  0001 C CNN
+F 2 "Capacitor_SMD:C_0805_2012Metric" H 1500 1750 50  0001 C CNN
 F 3 "~" H 1500 1750 50  0001 C CNN
 	1    1500 1750
@@
 F 0 "C?" H 11092 2596 50  0000 L CNN
 F 1 "22pF" H 11092 2505 50  0000 L CNN
-F 2 "" H 11000 2550 50  0001 C CNN
+F 2 "Capacitor_SMD:C_0805_2012Metric" H 11000 2550 50  0001 C CNN
 F 3 "~" H 11000 2550 50  0001 C CNN
 	1    11000 2550
@@
 F 0 "D?" H 10050 745 50  0000 C CNN
 F 1 "LED_green" H 10050 836 50  0000 C CNN
-F 2 "" V 10050 950 50  0001 C CNN
+F 2 "LED_SMD:LED_1206_3216Metric" V 10050 950 50  0001 C CNN
 F 3 "~" V 10050 950 50  0001 C CNN
 	1    10050 950
@@
 F 0 "C?" H 11642 1196 50  0000 L CNN
 F 1 "10uF" H 11642 1105 50  0000 L CNN
-F 2 "" H 11550 1150 50  0001 C CNN
+F 2 "Capacitor_SMD:C_0805_2012Metric" H 11550 1150 50  0001 C CNN
 F 3 "~" H 11550 1150 50  0001 C CNN
 	1    11550 1150
@@
 F 0 "D?" H 8450 745 50  0000 C CNN
 F 1 "LED_RX_red" H 8450 836 50  0000 C CNN
-F 2 "" V 8450 950 50  0001 C CNN
+F 2 "LED_SMD:LED_1206_3216Metric" V 8450 950 50  0001 C CNN
 F 3 "~" V 8450 950 50  0001 C CNN
 	1    8450 950
@@
 F 0 "D?" H 8450 1150 50  0000 C CNN
 F 1 "LED_TX_red" H 8450 1250 50  0000 C CNN
-F 2 "" V 8450 1050 50  0001 C CNN
+F 2 "LED_SMD:LED_1206_3216Metric" V 8450 1050 50  0001 C CNN
 F 3 "~" V 8450 1050 50  0001 C CNN
 	1    8450 1050
@@
 F 0 "C?" H 15592 7846 50  0000 L CNN
 F 1 "100nF" H 15592 7755 50  0000 L CNN
-F 2 "" H 15500 7800 50  0001 C CNN
+F 2 "Capacitor_SMD:C_0805_2012Metric" H 15500 7800 50  0001 C CNN
 F 3 "~" H 15500 7800 50  0001 C CNN
 	1    15500 7800
@@
 F 0 "C?" H 13300 8150 50  0000 L CNN
 F 1 "100nF" H 13300 8000 50  0000 L CNN
-F 2 "" H 13550 8100 50  0001 C CNN
+F 2 "Capacitor_SMD:C_0805_2012Metric" H 13550 8100 50  0001 C CNN
 F 3 "~" H 13550 8100 50  0001 C CNN
 	1    13550 8100
@@
 F 0 "C?" V 12971 7100 50  0000 C CNN
 F 1 "C_Small" V 13062 7100 50  0000 C CNN
-F 2 "" H 13200 7100 50  0001 C CNN
+F 2 "Capacitor_SMD:C_0805_2012Metric" H 13200 7100 50  0001 C CNN
 F 3 "~" H 13200 7100 50  0001 C CNN
 	1    13200 7100
@@
 F 0 "C?" H 8092 10546 50  0000 L CNN
 F 1 "100nF" H 8092 10455 50  0000 L CNN
-F 2 "" H 8000 10500 50  0001 C CNN
+F 2 "Capacitor_SMD:C_0805_2012Metric" H 8000 10500 50  0001 C CNN
 F 3 "~" H 8000 10500 50  0001 C CNN
 	1    8000 10500
@@
 F 0 "C?" H 9542 3746 50  0000 L CNN
 F 1 "100nF" H 9542 3655 50  0000 L CNN
-F 2 "" H 9450 3700 50  0001 C CNN
+F 2 "Capacitor_SMD:C_0805_2012Metric" H 9450 3700 50  0001 C CNN
 F 3 "~" H 9450 3700 50  0001 C CNN
 	1    9450 3700

Commit message: Footprints für Widerstände
Parts:
- R? (x30): footprint (none) -> Resistor_SMD:R_0805_2012Metric
Changed lines of the file:
@@
 F 0 "R?" H 750 1450 50  0000 L CNN
 F 1 "1M" H 750 1250 50  0000 L CNN
-F 2 "" H 900 1350 50  0001 C CNN
+F 2 "Resistor_SMD:R_0805_2012Metric" H 900 1350 50  0001 C CNN
 F 3 "~" H 900 1350 50  0001 C CNN
 	1    900  1350
@@
 F 0 "R?" V 8054 2550 50  0000 C CNN
 F 1 "10K" V 8150 2550 50  0000 C CNN
-F 2 "" H 8250 2550 50  0001 C CNN
+F 2 "Resistor_SMD:R_0805_2012Metric" H 8250 2550 50  0001 C CNN
 F 3 "~" H 8250 2550 50  0001 C CNN
 	1    8250 2550
@@
 F 0 "R?" V 8150 2650 50  0000 C CNN
 F 1 "10K" V 8050 2650 50  0000 C CNN
-F 2 "" H 8250 2650 50  0001 C CNN
+F 2 "Resistor_SMD:R_0805_2012Metric" H 8250 2650 50  0001 C CNN
 F 3 "~" H 8250 2650 50  0001 C CNN
 	1    8250 2650
@@
 F 0 "R?" H 11059 2396 50  0000 L CNN
 F 1 "10K" H 11059 2305 50  0000 L CNN
-F 2 "" H 11000 2350 50  0001 C CNN
+F 2 "Resistor_SMD:R_0805_2012Metric" H 11000 2350 50  0001 C CNN
 F 3 "~" H 11000 2350 50  0001 C CNN
 	1    11000 2350
@@
 F 0 "R?" V 9454 950 50  0000 C CNN
 F 1 "1K" V 9545 950 50  0000 C CNN
-F 2 "" H 9650 950 50  0001 C CNN
+F 2 "Resistor_SMD:R_0805_2012Metric" H 9650 950 50  0001 C CNN
 F 3 "~" H 9650 950 50  0001 C CNN
 	1    9650 950
@@
 F 0 "R?" H 13109 1146 50  0000 L CNN
 F 1 "10K" H 13109 1055 50  0000 L CNN
-F 2 "" H 13050 1100 50  0001 C CNN
+F 2 "Resistor_SMD:R_0805_2012Metric" H 13050 1100 50  0001 C CNN
 F 3 "~" H 13050 1100 50  0001 C CNN
 	1    13050 1100
@@
 F 0 "R?" H 14709 1146 50  0000 L CNN
 F 1 "10K" H 14709 1055 50  0000 L CNN
-F 2 "" H 14650 1100 50  0001 C CNN
+F 2 "Resistor_SMD:R_0805_2012Metric" H 14650 1100 50  0001 C CNN
 F 3 "~" H 14650 1100 50  0001 C CNN
 	1    14650 1100
@@
 F 0 "R?" H 13109 1996 50  0000 L CNN
 F 1 "10K" H 13109 1905 50  0000 L CNN
-F 2 "" H 13050 1950 50  0001 C CNN
+F 2 "Resistor_SMD:R_0805_2012Metric" H 13050 1950 50  0001 C CNN
 F 3 "~" H 13050 1950 50  0001 C CNN
 	1    13050 1950
@@
 F 0 "R?" H 14709 1996 50  0000 L CNN
 F 1 "10K" H 14709 1905 50  0000 L CNN
-F 2 "" H 14650 1950 50  0001 C CNN
+F 2 "Resistor_SMD:R_0805_2012Metric" H 14650 1950 50  0001 C CNN
 F 3 "~" H 14650 1950 50  0001 C CNN
 	1    14650 1950
@@
 F 0 "R?" H 14809 4846 50  0000 L CNN
 F 1 "10K" V 14850 4650 50  0000 L CNN
-F 2 "" H 14750 4800 50  0001 C CNN
+F 2 "Resistor_SMD:R_0805_2012Metric" H 14750 4800 50  0001 C CNN
 F 3 "~" H 14750 4800 50  0001 C CNN
 	1    14750 4800
@@
 F 0 "R?" H 14509 4746 50  0000 L CNN
 F 1 "10K" V 14550 4550 50  0000 L CNN
-F 2 "" H 14450 4700 50  0001 C CNN
+F 2 "Resistor_SMD:R_0805_2012Metric" H 14450 4700 50  0001 C CNN
 F 3 "~" H 14450 4700 50  0001 C CNN
 	1    14450 4700
@@
 F 0 "R?" H 14209 4646 50  0000 L CNN
 F 1 "10K" V 14250 4450 50  0000 L CNN
-F 2 "" H 14150 4600 50  0001 C CNN
+F 2 "Resistor_SMD:R_0805_2012Metric" H 14150 4600 50  0001 C CNN
 F 3 "~" H 14150 4600 50  0001 C CNN
 	1    14150 4600
@@
 F 0 "R?" H 13909 4546 50  0000 L CNN
 F 1 "10K" V 13950 4350 50  0000 L CNN
-F 2 "" H 13850 4500 50  0001 C CNN
+F 2 "Resistor_SMD:R_0805_2012Metric" H 13850 4500 50  0001 C CNN
 F 3 "~" H 13850 4500 50  0001 C CNN
 	1    13850 4500
@@
 F 0 "R?" H 13559 4446 50  0000 L CNN
 F 1 "10K" V 13600 4250 50  0000 L CNN
-F 2 "" H 13500 4400 50  0001 C CNN
+F 2 "Resistor_SMD:R_0805_2012Metric" H 13500 4400 50  0001 C CNN
 F 3 "~" H 13500 4400 50  0001 C CNN
 	1    13500 4400
@@
 F 0 "R?" H 13259 4346 50  0000 L CNN
 F 1 "10K" V 13300 4150 50  0000 L CNN
-F 2 "" H 13200 4300 50  0001 C CNN
+F 2 "Resistor_SMD:R_0805_2012Metric" H 13200 4300 50  0001 C CNN
 F 3 "~" H 13200 4300 50  0001 C CNN
 	1    13200 4300
@@
 F 0 "R?" H 8209 8546 50  0000 L CNN
 F 1 "10K" H 8209 8455 50  0000 L CNN
-F 2 "" H 8150 8500 50  0001 C CNN
+F 2 "Resistor_SMD:R_0805_2012Metric" H 8150 8500 50  0001 C CNN
 F 3 "~" H 8150 8500 50  0001 C CNN
 	1    8150 8500
@@
 F 0 "R?" H 7550 8550 50  0000 L CNN
 F 1 "10K" H 7550 8450 50  0000 L CNN
-F 2 "" H 7750 8500 50  0001 C CNN
+F 2 "Resistor_SMD:R_0805_2012Metric" H 7750 8500 50  0001 C CNN
 F 3 "~" H 7750 8500 50  0001 C CNN
 	1    7750 8500
@@
 F 0 "R?" H 9359 8546 50  0000 L CNN
 F 1 "10K" H 9359 8455 50  0000 L CNN
-F 2 "" H 9300 8500 50  0001 C CNN
+F 2 "Resistor_SMD:R_0805_2012Metric" H 9300 8500 50  0001 C CNN
 F 3 "~" H 9300 8500 50  0001 C CNN
 	1    9300 8500
@@
 F 0 "R?" H 8700 8550 50  0000 L CNN
 F 1 "10K" H 8700 8450 50  0000 L CNN
-F 2 "" H 8900 8500 50  0001 C CNN
+F 2 "Resistor_SMD:R_0805_2012Metric" H 8900 8500 50  0001 C CNN
 F 3 "~" H 8900 8500 50  0001 C CNN
 	1    8900 8500
@@
 F 0 "R?" H 8559 5196 50  0000 L CNN
 F 1 "10K" H 8559 5105 50  0000 L CNN
-F 2 "" H 8500 5150 50  0001 C CNN
+F 2 "Resistor_SMD:R_0805_2012Metric" H 8500 5150 50  0001 C CNN
 F 3 "~" H 8500 5150 50  0001 C CNN
 	1    8500 5150
@@
 F 0 "R?" H 7900 5200 50  0000 L CNN
 F 1 "10K" H 7900 5100 50  0000 L CNN
-F 2 "" H 8100 5150 50  0001 C CNN
+F 2 "Resistor_SMD:R_0805_2012Metric" H 8100 5150 50  0001 C CNN
 F 3 "~" H 8100 5150 50  0001 C CNN
 	1    8100 5150
@@
 F 0 "R?" H 10409 5196 50  0000 L CNN
 F 1 "10K" H 10409 5105 50  0000 L CNN
-F 2 "" H 10350 5150 50  0001 C CNN
+F 2 "Resistor_SMD:R_0805_2012Metric" H 10350 5150 50  0001 C CNN
 F 3 "~" H 10350 5150 50  0001 C CNN
 	1    10350 5150
@@
 F 0 "R?" H 9750 5200 50  0000 L CNN
 F 1 "10K" H 9750 5100 50  0000 L CNN
-F 2 "" H 9950 5150 50  0001 C CNN
+F 2 "Resistor_SMD:R_0805_2012Metric" H 9950 5150 50  0001 C CNN
 F 3 "~" H 9950 5150 50  0001 C CNN
 	1    9950 5150
@@
 F 0 "R?" V 8950 1050 50  0000 C CNN
 F 1 "1K" V 9050 1050 50  0000 C CNN
-F 2 "" H 8850 1050 50  0001 C CNN
+F 2 "Resistor_SMD:R_0805_2012Metric" H 8850 1050 50  0001 C CNN
 F 3 "~" H 8850 1050 50  0001 C CNN
 	1    8850 1050
@@
 F 0 "R?" V 9050 950 50  0000 C CNN
 F 1 "1K" V 8950 950 50  0000 C CNN
-F 2 "" H 8850 950 50  0001 C CNN
+F 2 "Resistor_SMD:R_0805_2012Metric" H 8850 950 50  0001 C CNN
 F 3 "~" H 8850 950 50  0001 C CNN
 	1    8850 950
@@
 F 0 "R?" V 15304 7300 50  0000 C CNN
 F 1 "1K" V 15395 7300 50  0000 C CNN
-F 2 "" H 15500 7300 50  0001 C CNN
+F 2 "Resistor_SMD:R_0805_2012Metric" H 15500 7300 50  0001 C CNN
 F 3 "~" H 15500 7300 50  0001 C CNN
 	1    15500 7300
@@
 F 0 "R?" V 15400 7400 50  0000 C CNN
 F 1 "1K" V 15300 7400 50  0000 C CNN
-F 2 "" H 15500 7400 50  0001 C CNN
+F 2 "Resistor_SMD:R_0805_2012Metric" H 15500 7400 50  0001 C CNN
 F 3 "~" H 15500 7400 50  0001 C CNN
 	1    15500 7400
@@
 F 0 "R?" H 8209 9646 50  0000 L CNN
 F 1 "10K" H 8209 9555 50  0000 L CNN
-F 2 "" H 8150 9600 50  0001 C CNN
+F 2 "Resistor_SMD:R_0805_2012Metric" H 8150 9600 50  0001 C CNN
 F 3 "~" H 8150 9600 50  0001 C CNN
 	1    8150 9600
@@
 F 0 "R?" H 10059 10046 50  0000 L CNN
 F 1 "10K" H 10059 9955 50  0000 L CNN
-F 2 "" H 10000 10000 50  0001 C CNN
+F 2 "Resistor_SMD:R_0805_2012Metric" H 10000 10000 50  0001 C CNN
 F 3 "~" H 10000 10000 50  0001 C CNN
 	1    10000 10000
@@
 F 0 "R?" H 9650 10000 50  0000 L CNN
 F 1 "10K" H 9650 9900 50  0000 L CNN
-F 2 "" H 9850 9950 50  0001 C CNN
+F 2 "Resistor_SMD:R_0805_2012Metric" H 9850 9950 50  0001 C CNN
 F 3 "~" H 9850 9950 50  0001 C CNN
 	1    9850 9950

Commit message: Footprints für CP Kondensatoren hinzugefügt
Parts:
- C? (x2): footprint (none) -> Capacitor_SMD:CP_Elec_6.3x5.7
Changed lines of the file:
@@
 F 0 "C?" H 9188 3746 50  0000 L CNN
 F 1 "47uF" H 9188 3655 50  0000 L CNN
-F 2 "" H 9100 3700 50  0001 C CNN
+F 2 "Capacitor_SMD:CP_Elec_6.3x5.7" H 9100 3700 50  0001 C CNN
 F 3 "~" H 9100 3700 50  0001 C CNN
 	1    9100 3700
@@
 F 0 "C?" H 8338 4046 50  0000 L CNN
 F 1 "47uF" H 8338 3955 50  0000 L CNN
-F 2 "" H 8250 4000 50  0001 C CNN
+F 2 "Capacitor_SMD:CP_Elec_6.3x5.7" H 8250 4000 50  0001 C CNN
 F 3 "~" H 8250 4000 50  0001 C CNN
 	1    8250 4000

Commit message: Footprints für Push Buttons
Parts:
- SW? (x2): footprint (none) -> Button_Switch_SMD:SW_SPST_FSMSM
Changed lines of the file:
@@
 F 0 "SW?" H 10150 2735 50  0000 C CNN
 F 1 "SW_Reset" H 10150 2644 50  0000 C CNN
-F 2 "" H 10150 2650 50  0001 C CNN
+F 2 "Button_Switch_SMD:SW_SPST_FSMSM" H 10150 2650 50  0001 C CNN
 F 3 "" H 10150 2650 50  0001 C CNN
 	1    10150 2450
@@
 F 0 "SW?" H 7800 9985 50  0000 C CNN
 F 1 "SW_ESP_Reset" H 7800 9894 50  0000 C CNN
-F 2 "" H 7800 9900 50  0001 C CNN
+F 2 "Button_Switch_SMD:SW_SPST_FSMSM" H 7800 9900 50  0001 C CNN
 F 3 "" H 7800 9900 50  0001 C CNN
 	1    7800 9700

Commit message: Diverse Footprints hinzugefügt
Parts:
- D? (x2): footprint (none) -> Diode_SMD:D_0805_2012Metric
- F?: footprint (none) -> Fuse:Fuse_1812_4532Metric
- Y?: footprint (none) -> Crystal:Resonator_SMD-3Pin_7.2x3.0mm
Changed lines of the file:
@@
 F 0 "Y?" V 1250 1500 50  0000 C CNN
 F 1 "CSTCE16M0V53-R0" V 1300 1850 50  0000 C CNN
-F 2 "" H 1275 1350 50  0001 C CNN
+F 2 "Crystal:Resonator_SMD-3Pin_7.2x3.0mm" H 1275 1350 50  0001 C CNN
 F 3 "~" H 1275 1350 50  0001 C CNN
 	1    1300 1350
@@
 F 0 "D?" V 11404 2418 50  0000 L CNN
 F 1 "CD1206-S01575" V 11495 2418 50  0000 L CNN
-F 2 "" V 11450 2350 50  0001 C CNN
+F 2 "Diode_SMD:D_0805_2012Metric" V 11450 2350 50  0001 C CNN
 F 3 "~" V 11450 2350 50  0001 C CNN
 	1    11450 2350
@@
 F 0 "F?" H 13068 7346 50  0000 L CNN
 F 1 "Poly 500mA" H 13068 7255 50  0000 L CNN
-F 2 "" H 13050 7100 50  0001 L CNN
+F 2 "Fuse:Fuse_1812_4532Metric" H 13050 7100 50  0001 L CNN
 F 3 "~" H 13000 7300 50  0001 C CNN
 	1    13000 7300
@@
 F 0 "D?" H 9850 3395 50  0000 C CNN
 F 1 "M7" H 9850 3486 50  0000 C CNN
-F 2 "" V 9850 3600 50  0001 C CNN
+F 2 "Diode_SMD:D_0805_2012Metric" V 9850 3600 50  0001 C CNN
 F 3 "~" V 9850 3600 50  0001 C CNN
 	1    9850 3600
