File: PCB/TaggerKeypadDisplay/TaggerKeypadDisplay.kicad_pcb (KiCad board)
At the start: 2 copper layers, 35 parts, among them J1 JST_PH_Keypad, J2 JST_PH_Display, Q1 BSS138, Q2 BSS138, SW1 key_up, SW2 key_down, SW3 key_left, SW4 key_right, SW5 key_back, SW6 key_enter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

Commit message: Anpassungen
Parts:
- D1, D2, D3: footprint Diode_SMD:D_0805_2012Metric -> Diode_SMD:D_SOD-123
- moved D1 5.40 mm to (57.4, 61.2)
- moved U2 3.60 mm to (49.0, 40.4)
- moved SW5 3.00 mm to (63.4, 63.8), turned to 90 degrees
- moved SW6 3.00 mm to (34.6, 63.8), turned to 90 degrees
- moved D3 2.45 mm to (55.2, 56.4), turned to 0 degrees
- moved D2 0.67 mm to (50.4, 55.6)
Routing:
- net GND: track 53.4 -> 104.4 mm
- net +5V: track 105.6 -> 121.5 mm
- net CS_3.3V: track 17.3 -> 26.3 mm
- net +3V3: track 64.5 -> 71.7 mm
- net D1-MOSI-SDA_3.3V: track 45.0 -> 51.5 mm
- net DC-SA0_3.3V: track 17.8 -> 24.2 mm
- net key_back: track 23.3 -> 28.9 mm
- net display_SJ2: track 66.7 -> 71.2 mm
- net Net-(JP2-Pad1): track 13.0 -> 17.2 mm
- net Net-(C8-Pad1): track 4.13 -> 7.93 mm
- net Net-(C3-Pad1): track 4.62 -> 8.42 mm
- net Net-(C7-Pad1): track 5.24 -> 8.84 mm
- net Net-(C4-Pad2): track 4.95 -> 8.55 mm
- net Net-(C4-Pad1): track 4.46 -> 8.06 mm
- net Net-(C3-Pad2): track 4.13 -> 7.73 mm
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Other:
- board text added: "Keypad V3/04.19/10 www.infinitag.io"
- board text removed: "Keypad V2/03.19/10 www.infinitag.io"
- board text removed: "|Infinitag"

Commit message: Updates
Other:
- board outline added: 38 x 59 mm
Changed lines of the file:
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@@
   (general
     (thickness 1.6)
-    (drawings 17)
+    (drawings 10)
     (tracks 403)
     (zones 0)
@@
   )
   (setup
-    (last_trace_width 0.4)
+    (last_trace_width 0.2)
     (user_trace_width 0.2)
     (user_trace_width 0.4)
@@
       (usegerberadvancedattributes false)
       (creategerberjobfile false)
-      (excludeedgelayer true)
+      (excludeedgelayer false)
       (linewidth 0.100000)
       (plotframeref false)
@@
     )
   )
+  (gr_line (start 68 30) (end 56 30) (layer Edge.Cuts) (width 0.15))
+  (gr_line (start 68 89) (end 68 30) (layer Edge.Cuts) (width 0.15))
+  (gr_line (start 30 89) (end 68 89) (layer Edge.Cuts) (width 0.15))
+  (gr_line (start 30 30) (end 30 89) (layer Edge.Cuts) (width 0.15))
+  (gr_line (start 42 30) (end 30 30) (layer Edge.Cuts) (width 0.15))
+  (gr_line (start 42 34) (end 42 30) (layer Edge.Cuts) (width 0.15))
+  (gr_line (start 56 34) (end 42 34) (layer Edge.Cuts) (width 0.15))
+  (gr_line (start 56 30) (end 56 34) (layer Edge.Cuts) (width 0.15))
   (gr_text "Keypad V3/04.19/10\nwww.infinitag.io" (at 44 86.2) (layer F.SilkS)
     (effects (font (size 1 1) (thickness 0.1)) (justify left))
@@
     (effects (font (size 1.5 1.5) (thickness 0.2)) (justify left))
   )
-  (gr_line (start 30 89) (end 30 62) (layer F.SilkS) (width 0.2))
-  (gr_line (start 49 89) (end 30 89) (layer F.SilkS) (width 0.2))
-  (gr_line (start 68 89) (end 49 89) (layer F.SilkS) (width 0.2))
-  (gr_line (start 68 63) (end 68 89) (layer F.SilkS) (width 0.2))
-  (gr_line (start 30 35) (end 30 62) (layer F.SilkS) (width 0.2))
-  (gr_line (start 68 36) (end 68 63) (layer F.SilkS) (width 0.2))
-  (gr_line (start 42 34) (end 42 33) (layer F.SilkS) (width 0.2))
-  (gr_line (start 56 34) (end 42 34) (layer F.SilkS) (width 0.2))
-  (gr_line (start 56 30) (end 56 34) (layer F.SilkS) (width 0.2))
-  (gr_line (start 42 30) (end 30 30) (layer F.SilkS) (width 0.2))
-  (gr_line (start 68 30) (end 56 30) (layer F.SilkS) (width 0.2))
-  (gr_line (start 56 33) (end 56 30) (layer F.SilkS) (width 0.2))
-  (gr_line (start 42 30) (end 42 33) (layer F.SilkS) (width 0.2))
-  (gr_line (start 30 30) (end 30 35) (layer F.SilkS) (width 0.2))
-  (gr_line (start 68 30) (end 68 36) (layer F.SilkS) (width 0.2))
   (segment (start 47.8 76.9) (end 46.65 76.9) (width 0.4) (layer F.Cu) (net 1))
   (segment (start 44 74.25) (end 44 71.5) (width 0.4) (layer F.Cu) (net 1))

Commit message: Updates
Routing:
- net +5V: track 121.5 -> 136.2 mm, vias 4 -> 5
- net key_enter: track 62.0 -> 71.9 mm
- net key_down: track 21.1 -> 30.6 mm
- net key_left: track 13.9 -> 22.3 mm, vias 0 -> 2
- net key_back: track 28.9 -> 36.6 mm
- net key_right: track 35.0 -> 27.9 mm
- net key_up: track 12.2 -> 15.7 mm
