File: PCB/TaggerMainboard_schmal/TaggerMainboard.sch (KiCad schematic (older format))
At the start: 62 parts, among them J1 VIN, J10 JST_PH_Info, J11 JST_PH_LEDbar_right, J12 JST_PH_IrLED, J13 JST_PH_Reload, J14 JST_PH_Special, J15 JST_PH_LEDbar_left, J16 JSP_PH_Sensor, J17 Infinitag_Shield, J18 JST_PH_Keypad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

Commit message: Updates
Parts:
- removed J2: JST_PH_Speaker, Connector_JST:JST_PH_B2B-PH-K_1x02_P2.00mm_Vertical, symbol Connector_Generic:Conn_01x02
- removed U6: FT232RL, Package_SO:SSOP-28_5.3x10.2mm_P0.65mm, symbol Interface_USB:FT232RL
- added C15: 1u, Capacitor_SMD:C_0805_2012Metric, symbol Device:C_Small
- added C16: 100n, Capacitor_SMD:C_0805_2012Metric, symbol Device:C_Small
- added C17: 100nF, Capacitor_SMD:C_0805_2012Metric, symbol Device:C_Small
- added D6, D7: CG0603MLC-05E, Diode_SMD:D_0603_1608Metric, symbol Device:D_TVS
- added D8: CD1206-S01575, Diode_SMD:D_1206_3216Metric, symbol Device:D_Small
- added FB1: BLM21PG 221, Inductor_SMD:L_0805_2012Metric, symbol Device:Ferrite_Bead_Small
- added J19: Conn_02x03_Odd_Even, Infinitag:ICSP_Pogo, symbol Connector_Generic:Conn_02x03_Odd_Even
- added J2: JST_PH_Speaker, Connector_JST:JST_PH_B4B-PH-K_1x04_P2.00mm_Vertical, symbol Connector_Generic:Conn_01x04
- added JP1: SolderJumper_2_Bridged, Jumper:SolderJumper-2_P1.3mm_Bridged_Pad1.0x1.5mm, symbol Jumper:SolderJumper_2_Bridged
- added RN4: 22R, Resistor_SMD:R_Array_Convex_4x0603, symbol Device:R_Pack04
- added RN5: 1K, Resistor_SMD:R_Array_Convex_4x0603, symbol Device:R_Pack04
- added U6: ATmega16U2-MU, Package_DFN_QFN:QFN-32-1EP_5x5mm_P0.5mm_EP3.1x3.1mm, symbol MCU_Microchip_ATmega:ATmega16U2-MU
- added Y2: 16MHz, Crystal:Crystal_SMD_HC49-SD, symbol Device:Crystal_Small
- C11: value 100nF -> 100n
- C12, C14: value 100nF -> 22p
- J6: footprint Connector_PinHeader_2.54mm:PinHeader_2x03_P2.54mm_Vertical -> Infinitag:ICSP_Pogo
- R10: value 1K -> 1M
- R11: value 1K -> 10K
Connections:
- net +5V: now also R11.2, C16.2, D8.1 (K), J19.2 (Pin_2), U6.32 (AVCC), U6.4 (VCC); no longer C12.1
- net GND: now also C14.2, C16.1, J19.6 (Pin_6), J2.2 (Pin_2), J2.4 (Pin_4), JP1.2 (B), RN5.5 (R4.2), U6.3 (GND), U6.33 (GND); no longer J5.5 (GND), J5.6 (Shield)
- net LED_RX: now also U6.10 (PD4)
- net LED_TX: now also U6.11 (PD5)
- net RESET: now also C17.1; no longer C14.2
- net RX0: now also RN5.7 (R2.2); no longer R10.1
- net TX0: now also RN5.8 (R1.2); no longer R11.2
- net VBUS: now also U6.31 (UVCC)
- net at R10.2: now also C14.1, U6.2 (PC0/XTAL2), Y2.2
- net at J5.3 (D+): now also D6.1 (A1), RN4.1 (R1.1)
- net at J5.2 (D-): now also D7.1 (A1), RN4.2 (R2.1)
- net at R11.1: now also D8.2 (A), J19.5 (Pin_5), U6.24 (PC1/~RESET)
- net at J5.4 (ID): now also C15.2, FB1.1, JP1.1 (A), U6.28 (UGND)
- net DF_SPK+ renamed DF_SPK_LEFT
- net DF_SPK_LEFT: now also J2.1 (Pin_1)
- net DF_SPK- renamed DF_SPK_RIGHT
- net DF_SPK_RIGHT: now also J2.3 (Pin_3)
- new net: C12.1, R10.1, U6.1 (XTAL1), Y2.1
- new net: C17.2, RN5.4 (R4.1), U6.13 (~HWB~/PD7)
- new net: J19.4 (Pin_4), U6.15 (PB1)
- new net: J19.1 (Pin_1), U6.16 (PB2)
- new net: J19.3 (Pin_3), U6.17 (PB3)
- new net: C15.1, U6.27 (UCAP)
- new net: RN4.7 (R2.2), U6.29 (D+)
- new net: RN4.8 (R1.2), U6.30 (D-)
- new net: RN5.1 (R1.1), U6.8 (PD2)
- new net: RN5.2 (R2.1), U6.9 (PD3)
- new net: D6.2 (A2), D7.2 (A2), FB1.2, J5.5 (GND), J5.6 (Shield)
- no-connect marks 74 -> 81
Other:
- moved on the sheet: C1, C2, C3, C4, C5, C6, C8, D4, J1, J4, L1, Q1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
